File: hardware/kicad/the_harp/ADC Driver.kicad_sch (KiCad schematic)
At the start: 17 parts, among them U601 THS4522IPW

Commit message: Input buffer: OPA2365 and the Timekeeper's H2 fix
The OPA1656's input range ends at (V+) - 2.25 V, 2.75 V on the 5 V rail,
0.25 V above the 2.5 V bias, while hard-played guitar peaks reach about
+/-1.5 V at the buffer (from the Timekeeper's measured levels). U701 becomes
an OPA2365 (zero-crossover rail-to-rail input, 2.2-5.5 V, pin-compatible),
so the bias, the THS4522 and the 5 V rail stay as they are.

H2 from the Timekeeper's input noise review: R705 5k1 -> 49.9R and
R602 1k -> 1.05k, so the THS4522 runs at gain 1 with balanced legs.
Docs record the decision and the matching Timekeeper rework.

Co-Authored-By: Claude Opus 5.5 <noreply@anthropic.com>
Claude-Session: https://claude.ai/code/session_01ToUUHuo6mg178NkLtQkDLg
Parts:
- R602: value 1k -> 1.05k
Changed lines of the file:
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@@
 			)
 		)
-		(property "Value" "1k"
+		(property "Value" "1.05k"
 			(at 208.28 55.84 0)
 			(show_name no)
@@
 			)
 		)
-		(property "Description" ""
+		(property "Description" "= R601 + R705: matches the signal leg (Timekeeper review H2)"
 			(at 205.74 48.26 0)
 			(hide yes)

Commit message: ADC driver gain 0.59: R603/R604 620R
Same choice as the Timekeeper: at 620R a 4.8 Vpp input, the most the
OPA2365 buffer can swing on 5 V, just reaches ADC full scale, so guitar and
synth both reach the ADC cleanly. Docs updated; merges main (firmware
requirements draft) with the README conflict resolved.

Co-Authored-By: Claude Opus 5.5 <noreply@anthropic.com>
Claude-Session: https://claude.ai/code/session_01ToUUHuo6mg178NkLtQkDLg
Parts:
- R603, R604: value 1k -> 620
Other:
- note added: "Single-ended to differential ADC driver, the Timekeeper's AnalogInputBuffer: THS4522 channel A, gain 0.59 (620R / 1.05k), 40.2R + 2.7n differential filter, VOCM from VCOM_B. The input reference (INN side) goes to VCOM_A, the DC level of the input buffer output (the Timekeeper left it open). Channel B is powered down [CONFIRM unused-channel handling in the THS4522 datasheet]."
- note removed: "Single-ended to differential ADC driver, the Timekeeper's AnalogInputBuffer: THS4522 channel A, gain 1 (1k/1k), 40.2R + 2.7n differential filter, VOCM from VCOM_B. The input reference (INN side) goes to VCOM_A, the DC level of the input buffer output (the Timekeeper left it open). Channel B is powered down [CONFIRM unused-channel handling in the THS4522 datasheet]."
Changed lines of the file:
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@@
 			)
 		)
-		(property "Value" "1k"
+		(property "Value" "620"
 			(at 226.06 58.38 0)
 			(show_name no)
@@
 			)
 		)
-		(property "Description" ""
+		(property "Description" "gain 0.59: a 4.8 Vpp input just reaches ADC full scale"
 			(at 223.52 50.8 0)
 			(hide yes)
@@
 			)
 		)
-		(property "Value" "1k"
+		(property "Value" "620"
 			(at 261.62 58.38 0)
 			(show_name no)
@@
 			)
 		)
-		(property "Description" ""
+		(property "Description" "gain 0.59: a 4.8 Vpp input just reaches ADC full scale"
 			(at 259.08 50.8 0)
 			(hide yes)
@@
 		)
 	)
-	(text "Single-ended to differential ADC driver, the Timekeeper's AnalogInputBuffer: THS4522 channel A, gain 1 (1k/1k), 40.2R + 2.7n differential filter, VOCM from VCOM_B.\nThe input reference (INN side) goes to VCOM_A, the DC level of the input buffer output (the Timekeeper left it open). Channel B is powered down [CONFIRM unused-channel handling in the THS4522 datasheet]."
+	(text "Single-ended to differential ADC driver, the Timekeeper's AnalogInputBuffer: THS4522 channel A, gain 0.59 (620R / 1.05k), 40.2R + 2.7n differential filter, VOCM from VCOM_B.\nThe input reference (INN side) goes to VCOM_A, the DC level of the input buffer output (the Timekeeper left it open). Channel B is powered down [CONFIRM unused-channel handling in the THS4522 datasheet]."
 		(exclude_from_sim no)
 		(at 20.32 15.24 0)
