File: hardware/kicad/the_harp/Analog In and Out.kicad_sch (KiCad schematic)
At the start: 26 parts, among them U701 OPA1656IDR, U702 OPA1688IDR

Commit message: Drop the THS4522: drive the ADC from the input OPA1656
The spare half of the input OPA1656 becomes a unity inverter about VCOM_A,
so U701A drives AINL+ and U701B drives AINL- through the THS4522 stage's
own output filter (40.2R per leg, 2.7n across, 100p to GND). Removes the
ADC Driver sheet (THS4522 and 16 passives) and, with it, the Timekeeper's
floating IN_N defect. 6 sheets, 183 parts, net check clean.

Co-Authored-By: Claude Opus 5.5 <noreply@anthropic.com>
Claude-Session: https://claude.ai/code/session_01ToUUHuo6mg178NkLtQkDLg
Parts:
- added C708, C709, C710: 100p, Capacitor_SMD:C_0603_1608Metric, symbol Device:C
- added R712: 10k, Resistor_SMD:R_0603_1608Metric, symbol Device:R
- added R713, R720: 40.2, Resistor_SMD:R_0603_1608Metric, symbol Device:R
- C702: value 220p -> 2.7n
- R705: value 5k1 -> 10k
Connections:
- net GND: now also C709.2, C710.2; no longer C702.2
- net IN_BUF_OUT: now also R713.1
- net EFFECT_IN_BUF renamed ADC_P
- net ADC_P: now also C709.1, R713.2; no longer R705.2
- net U701B_OUT renamed INV_FB
- net INV_FB: now also R705.2, C708.1, R712.1; no longer U701.7
- new net ADC_N: C702.2, C710.1, R720.2
- new net INV_OUT: C708.2, R712.2, R720.1, U701.7
Other:
- note added: "Input buffer and ADC drive (U701, OPA1656) and output stages (U702, OPA1688), the Timekeeper's ANALOG_FRONT on one 5 V rail biased at VCOM. In: 1M to ground at the relay, 100n film, 1M bias to VCOM_A, follower U701A (R703 0R; R704 + C707 to VCOM_A, both DNP, set gain). ADC drive without the Timekeeper's THS4522: U701A drives AINL+, U701B (unity inverter about VCOM_A, 10k/10k) drives AINL-; 40.2R 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"
- note removed: "Input buffer (U701A, OPA1656) and output stages (U702, OPA1688), the Timekeeper's ANALOG_FRONT on one 5 V rail biased at VCOM. In: 1M to ground at the relay, 100n film, 1M bias to VCOM_A, follower (R703 0R; R704 + C707 to VCOM_A, both DNP, set gain), 5k1 / 220p to the ADC driver. Out: unity-gain difference amplifier per channel (10k x4) referenced to VCOM_B, 10u out, 100R series, 1M pull-down."
- moved on the sheet: C702, C703, C704, C705, C706, C707, R703, R704, R705, R706, R707, R708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

Commit message: Restore the THS4522 ADC driver
Reverts c744d80. The THS4522 is designed for the single 5 V analog rail
(rail-to-rail output, VOCM sets the output common mode at the codec's VCOM),
which is why the Timekeeper uses it; the OPA1656 sits at the bottom of its
supply range there. The reference leg stays tied to VCOM_A, the fix from the
Timekeeper's input noise review (H1), not left floating.

Co-Authored-By: Claude Opus 5.5 <noreply@anthropic.com>
Claude-Session: https://claude.ai/code/session_01ToUUHuo6mg178NkLtQkDLg
Parts:
- removed C708, C709, C710: 100p, Capacitor_SMD:C_0603_1608Metric, symbol Device:C
- removed R712: 10k, Resistor_SMD:R_0603_1608Metric, symbol Device:R
- removed R713, R720: 40.2, Resistor_SMD:R_0603_1608Metric, symbol Device:R
- C702: value 2.7n -> 220p
- R705: value 10k -> 5k1
Connections:
- net ADC_N is gone; now on net GND: C702.2
- net INV_OUT is gone; now on net U701B_OUT: U701.7
- net ADC_P renamed EFFECT_IN_BUF
- net EFFECT_IN_BUF: now also R705.2
- net INV_FB renamed U701B_OUT
- net U701B_OUT: no longer R705.2
Other:
- note added: "Input buffer (U701A, OPA1656) and output stages (U702, OPA1688), the Timekeeper's ANALOG_FRONT on one 5 V rail biased at VCOM. In: 1M to ground at the relay, 100n film, 1M bias to VCOM_A, follower (R703 0R; R704 + C707 to VCOM_A, both DNP, set gain), 5k1 / 220p to the ADC driver. Out: unity-gain difference amplifier per channel (10k x4) referenced to VCOM_B, 10u out, 100R series, 1M pull-down."
- note removed: "Input buffer and ADC drive (U701, OPA1656) and output stages (U702, OPA1688), the Timekeeper's ANALOG_FRONT on one 5 V rail biased at VCOM. In: 1M to ground at the relay, 100n film, 1M bias to VCOM_A, follower U701A (R703 0R; R704 + C707 to VCOM_A, both DNP, set gain). ADC drive without the Timekeeper's THS4522: U701A drives AINL+, U701B (unity inverter about VCOM_A, 10k/10k) drives AINL-; 40.2R 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"
- moved on the sheet: C702, C703, C704, C705, C706, C707, R703, R704, R705, R706, R707, R708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

Commit message: Input buffer: OPA2365 and the Timekeeper's H2 fix
The OPA1656's input range ends at (V+) - 2.25 V, 2.75 V on the 5 V rail,
0.25 V above the 2.5 V bias, while hard-played guitar peaks reach about
+/-1.5 V at the buffer (from the Timekeeper's measured levels). U701 becomes
an OPA2365 (zero-crossover rail-to-rail input, 2.2-5.5 V, pin-compatible),
so the bias, the THS4522 and the 5 V rail stay as they are.

H2 from the Timekeeper's input noise review: R705 5k1 -> 49.9R and
R602 1k -> 1.05k, so the THS4522 runs at gain 1 with balanced legs.
Docs record the decision and the matching Timekeeper rework.

Co-Authored-By: Claude Opus 5.5 <noreply@anthropic.com>
Claude-Session: https://claude.ai/code/session_01ToUUHuo6mg178NkLtQkDLg
Parts:
- R705: value 5k1 -> 49.9
- U701: value OPA1656IDR -> OPA2365AIDR; Mfg Part # OPA1656IDR -> OPA2365AIDR
Other:
- note added: "Input buffer (U701A, OPA2365) and output stages (U702, OPA1688), the Timekeeper's ANALOG_FRONT on one 5 V rail biased at VCOM. U701 is an OPA2365 (zero-crossover rail-to-rail input) instead of the Timekeeper's OPA1656, whose input stops at (V+) - 2.25 V = 2.75 V on 5 V, 0.25 V above the 2.5 V bias; hard-played guitar peaks reach about +/-1.5 V here. R705 is 49.9R, not 5k1 (Timekeeper review H2). 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"
- note removed: "Input buffer (U701A, OPA1656) and output stages (U702, OPA1688), the Timekeeper's ANALOG_FRONT on one 5 V rail biased at VCOM. In: 1M to ground at the relay, 100n film, 1M bias to VCOM_A, follower (R703 0R; R704 + C707 to VCOM_A, both DNP, set gain), 5k1 / 220p to the ADC driver. Out: unity-gain difference amplifier per channel (10k x4) referenced to VCOM_B, 10u out, 100R series, 1M pull-down."
Changed lines of the file:
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@@
 			)
 		)
-		(property "Value" "OPA1656IDR"
+		(property "Value" "OPA2365AIDR"
 			(at 99.06 49.49 0)
 			(show_name no)
@@
 			)
 		)
-		(property "Mfg Part #" "OPA1656IDR"
+		(property "Mfg Part #" "OPA2365AIDR"
 			(at 96.52 43.18 0)
 			(hide yes)
@@
 			)
 		)
-		(property "Value" "OPA1656IDR"
+		(property "Value" "OPA2365AIDR"
 			(at 154.94 49.49 0)
 			(show_name no)
@@
 			)
 		)
-		(property "Mfg Part #" "OPA1656IDR"
+		(property "Mfg Part #" "OPA2365AIDR"
 			(at 152.4 43.18 0)
 			(hide yes)
@@
 			)
 		)
-		(property "Value" "OPA1656IDR"
+		(property "Value" "OPA2365AIDR"
 			(at 195.58 59.65 0)
 			(show_name no)
@@
 			)
 		)
-		(property "Mfg Part #" "OPA1656IDR"
+		(property "Mfg Part #" "OPA2365AIDR"
 			(at 193.04 48.26 0)
 			(hide yes)
@@
 			)
 		)
-		(property "Value" "5k1"
+		(property "Value" "49.9"
 			(at 266.7 60.92 0)
 			(show_name no)
@@
 			)
 		)
-		(property "Description" ""
+		(property "Description" "isolates U701A from C702 + C601; was 5k1 (Timekeeper review H2)"
 			(at 264.16 53.34 0)
 			(hide yes)
@@
 		)
 	)
-	(text "Input buffer (U701A, OPA1656) and output stages (U702, OPA1688), the Timekeeper's ANALOG_FRONT on one 5 V rail biased at VCOM.\nIn: 1M to ground at the relay, 100n film, 1M bias to VCOM_A, follower (R703 0R; R704 + C707 to VCOM_A, both DNP, set gain), 5k1 / 220p to the ADC driver.\nOut: unity-gain difference amplifier per channel (10k x4) referenced to VCOM_B, 10u out, 100R series, 1M pull-down."
+	(text "Input buffer (U701A, OPA2365) and output stages (U702, OPA1688), the Timekeeper's ANALOG_FRONT on one 5 V rail biased at VCOM.\nU701 is an OPA2365 (zero-crossover rail-to-rail input) instead of the Timekeeper's OPA1656, whose input stops at (V+) - 2.25 V = 2.75 V on 5 V, 0.25 V above the 2.5 V bias; hard-played guitar peaks reach about +/-1.5 V here. R705 is 49.9R, not 5k1 (Timekeeper review H2).\nIn: 1M to ground at the relay, 100n film, 1M bias to VCOM_A, follower (R703 0R; R704 + C707 to VCOM_A, both DNP, set gain), 49.9R / 220p to the ADC driver.\nOut: unity-gain difference amplifier per channel (10k x4) referenced to VCOM_B, 10u out, 100R series, 1M pull-down."
 		(exclude_from_sim no)
 		(at 20.32 15.24 0)
