File: hardware/kicad/the_harp/Controls and LEDs.kicad_sch (KiCad schematic)
At the start: 45 parts, among them SW101 Snap/Glide, SW102 Bypass mode, SW103 Exp target

Commit message: Follow The Alchemist's shared parts: NMJ6HCD2 jacks, G6K-2F-Y relay, JLCPCB numbers
- Jacks: Neutrik NMJ6HCD2 (JLCPCB HOOYA PJ-609BA, C309277); IN jack ring to
  GND as The Alchemist. PCB footprints copied from The Alchemist at its
  positions (origins 0.75/0.885 mm moved, nose axes unchanged).
- Relay: Omron G6K-2F-Y DC5 (C2982926), Alchemist pinout; PCB footprint at
  its position.
- Design and JLCPCB part numbers on the pots, relay drivers, LED drivers,
  footswitch RC, DC jack and the 5 V LDO; panel LEDs Kingbright WP710A10ID,
  dnp; footswitches on R2816 hand-solder pads, dnp.
- Docs: design brief decision 12, toggle conflict re-checked for the new
  jack geometry, stale OPA1656 mentions in pcb-plan corrected.
- Toggles not changed: The Alchemist's Taiway 100-DP6 is ON-ON-ON.

Co-Authored-By: Claude Opus 5.5 <noreply@anthropic.com>
Claude-Session: https://claude.ai/code/session_01ToUUHuo6mg178NkLtQkDLg
Parts:
- RV101, RV102, RV103, RV104, RV105, RV106: JLCPCB Manufacturer (none) -> Alpha (Taiwan); JLCPCB Part # (none) -> RD901F-40-15R1-B10K; LCSC (none) -> C20619174; Manufacturer (none) -> Alpha (Taiwan); Mfg Part # (none) -> RD901F-40-15R1-B10K; Supplier (none) -> LMS
