File: hardware/kicad/the_harp/Jacks and Bypass.kicad_sch (KiCad schematic)
At the start: 38 parts, among them J402 NRJ6HM-1, J403 NRJ6HM-1, J404 NRJ6HM-1, J405 Bypass FSW, J406 NRJ6HM-1, J407 Hold FSW, K401 EE2-5NU, Q401 2N7002, Q402 2N7002, Q403 2N7002, U401 MCP6001T-I/OT

Commit message: Follow The Alchemist's shared parts: NMJ6HCD2 jacks, G6K-2F-Y relay, JLCPCB numbers
- Jacks: Neutrik NMJ6HCD2 (JLCPCB HOOYA PJ-609BA, C309277); IN jack ring to
  GND as The Alchemist. PCB footprints copied from The Alchemist at its
  positions (origins 0.75/0.885 mm moved, nose axes unchanged).
- Relay: Omron G6K-2F-Y DC5 (C2982926), Alchemist pinout; PCB footprint at
  its position.
- Design and JLCPCB part numbers on the pots, relay drivers, LED drivers,
  footswitch RC, DC jack and the 5 V LDO; panel LEDs Kingbright WP710A10ID,
  dnp; footswitches on R2816 hand-solder pads, dnp.
- Docs: design brief decision 12, toggle conflict re-checked for the new
  jack geometry, stale OPA1656 mentions in pcb-plan corrected.
- Toggles not changed: The Alchemist's Taiway 100-DP6 is ON-ON-ON.

Co-Authored-By: Claude Opus 5.5 <noreply@anthropic.com>
Claude-Session: https://claude.ai/code/session_01ToUUHuo6mg178NkLtQkDLg
Parts:
- C408, C409: JLCPCB Manufacturer (none) -> YAGEO; JLCPCB Part # (none) -> CC0603KRX7R9BB104; LCSC (none) -> C14663; Manufacturer (none) -> YAGEO; Mfg Part # (none) -> CC0603KRX7R9BB104
- D113, D114: value LED -> RED_LED; Manufacturer (none) -> Kingbright; Mfg Part # (none) -> WP710A10ID; Supplier (none) -> Mouser; now not fitted
- D402: JLCPCB Manufacturer (none) -> hongjiacheng; JLCPCB Part # (none) -> 1N4148W; LCSC (none) -> C7420318; Manufacturer (none) -> Diodes Incorporated; Mfg Part # (none) -> 1N4148W-7-F
- J402, J403, J404, J406: value NRJ6HM-1 -> NMJ6HCD2; footprint Connector_Audio:Jack_6.35mm_Neutrik_NRJ6HM-1_Horizontal -> Connector_Audio:Jack_6.35mm_Neutrik_NMJ6HCD2_Horizontal; symbol Connector_Audio:NRJ6HM-1 -> Connector_Audio:NMJ6HCD2; JLCPCB Manufacturer (none) -> HOOYA; JLCPCB Part # (none) -> PJ-609BA; LCSC (none) -> C309277; Manufacturer (none) -> Neutrik; Mfg Part # (none) -> NMJ6HCD2; Supplier (none) -> JLCPCB
- J405, J407: footprint Connector_PinHeader_2.54mm:PinHeader_1x02_P2.54mm_Vertical -> Resistor_SMD:R_2816_7142Metric_Pad3.20x4.45mm_HandSolder; Supplier (none) -> none; now not fitted
- K401: value EE2-5NU -> G6K-2F-Y; footprint Relay_SMD:Relay_DPDT_Kemet_EE2_NU -> Relay_SMD:Relay_DPDT_Omron_G6K-2F-Y; symbol Relay:EE2-5NU -> Relay:G6K-2; JLCPCB Manufacturer (none) -> Omron Electronics; JLCPCB Part # (none) -> G6K-2F-Y-5V; LCSC (none) -> C2982926; Manufacturer KEMET -> Omron; Mfg Part # EE2-5NU -> G6K-2F-Y DC5; Supplier (none) -> JLCPCB
- Q401, Q402, Q403: JLCPCB Manufacturer (none) -> hongjiacheng; JLCPCB Part # (none) -> 2N7002; LCSC (none) -> C7420321; Manufacturer (none) -> onsemi; Mfg Part # (none) -> 2N7002LT1G
- R404, R410, R411, R414: JLCPCB Manufacturer (none) -> UNI ROYAL Uniroyal Elec; JLCPCB Part # (none) -> 0805W8F1001T5E; LCSC (none) -> C17513; Manufacturer (none) -> YAGEO; Mfg Part # (none) -> AC0805FR-071KL
- R405: JLCPCB Manufacturer (none) -> UNI ROYAL Uniroyal Elec; JLCPCB Part # (none) -> 1206W4F1500T5E; LCSC (none) -> C17917; Manufacturer (none) -> YAGEO; Mfg Part # (none) -> RC1206FR-07150RL; Supplier (none) -> JLCPCB
- R406, R408, R412: JLCPCB Manufacturer (none) -> FOJAN; JLCPCB Part # (none) -> FRQ0805F1000TS; LCSC (none) -> C7468571; Manufacturer (none) -> YAGEO; Mfg Part # (none) -> AC0805FR-07100RL
- R407, R409, R413: JLCPCB Manufacturer (none) -> UNI ROYAL Uniroyal Elec; JLCPCB Part # (none) -> 0805W8F1003T5E; LCSC (none) -> C149504; Manufacturer (none) -> YAGEO; Mfg Part # (none) -> AC0805FR-07100KL
Connections:
- net EFFECT_IN: now also K401.6; no longer K401.9
- net EFFECT_OUT_L: now also K401.4; no longer K401.5
- net GND: now also J402.R, K401.7; no longer K401.10
- net IN: now also K401.2, K401.5; no longer K401.3, K401.8
- net OUT_L: now also K401.3; no longer K401.4
- net RELAY_LOW: now also K401.8; no longer K401.12
- no-connect marks 15 -> 14
Other:
- note added: "Jacks on the Alchemist positions: IN (J402, right lower), EXP (J406, right upper), OUT L (J403, left lower), OUT R (J404, left upper). Relay true bypass after The Alchemist: K401 (Omron G6K-2F-Y, 5 V coil) at rest joins IN to OUT L (2-3) and grounds the effect input (6-7); energised it routes IN to the effect (5-6) and the effect to OUT L (3-4). IN jack ring to GND, as The Alchemist. OUT R is dri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"
- note removed: "Jacks on the Alchemist positions: IN (J402, right lower), EXP (J406, right upper), OUT L (J403, left lower), OUT R (J404, left upper). Relay true bypass after The Relic: K401 at rest joins IN to OUT L (3-4) and grounds the effect input (9-10); energised it routes IN to the effect (8-9) and the effect to OUT L (4-5). OUT R is driven straight from the DSP and is silent in true bypass; stereo player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"
