File: hardware/kicad/the_harp/Power.kicad_sch (KiCad schematic)
At the start: 24 parts, among them J401 PJ-063AH, U301 TPS54202DDC, U302 NCP718ASN500T1G

Commit message: Follow The Alchemist's shared parts: NMJ6HCD2 jacks, G6K-2F-Y relay, JLCPCB numbers
- Jacks: Neutrik NMJ6HCD2 (JLCPCB HOOYA PJ-609BA, C309277); IN jack ring to
  GND as The Alchemist. PCB footprints copied from The Alchemist at its
  positions (origins 0.75/0.885 mm moved, nose axes unchanged).
- Relay: Omron G6K-2F-Y DC5 (C2982926), Alchemist pinout; PCB footprint at
  its position.
- Design and JLCPCB part numbers on the pots, relay drivers, LED drivers,
  footswitch RC, DC jack and the 5 V LDO; panel LEDs Kingbright WP710A10ID,
  dnp; footswitches on R2816 hand-solder pads, dnp.
- Docs: design brief decision 12, toggle conflict re-checked for the new
  jack geometry, stale OPA1656 mentions in pcb-plan corrected.
- Toggles not changed: The Alchemist's Taiway 100-DP6 is ON-ON-ON.

Co-Authored-By: Claude Opus 5.5 <noreply@anthropic.com>
Claude-Session: https://claude.ai/code/session_01ToUUHuo6mg178NkLtQkDLg
Parts:
- J401: JLCPCB Manufacturer (none) -> CUI; JLCPCB Part # (none) -> PJ-063AH; LCSC (none) -> C22434582; Manufacturer CUI Devices -> Same Sky (formerly CUI Devices); Supplier (none) -> JLCPCB
- U302: JLCPCB Manufacturer (none) -> onsemi; JLCPCB Part # (none) -> NCP718ASN500T1G; LCSC (none) -> C603786
Changed lines of the file:
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@@
 			)
 		)
-		(property "Manufacturer" "CUI Devices"
+		(property "Manufacturer" "Same Sky (formerly CUI Devices)"
 			(at 38.1 40.64 0)
 			(hide yes)
@@
 			)
 		)
+		(property "LCSC" "C22434582"
+			(at 38.1 40.64 0)
+			(hide yes)
+			(show_name no)
+			(do_not_autoplace no)
+			(effects
+				(font
+					(size 1.27 1.27)
+				)
+			)
+		)
+		(property "JLCPCB Manufacturer" "CUI"
+			(at 38.1 40.64 0)
+			(hide yes)
+			(show_name no)
+			(do_not_autoplace no)
+			(effects
+				(font
+					(size 1.27 1.27)
+				)
+			)
+		)
+		(property "JLCPCB Part #" "PJ-063AH"
+			(at 38.1 40.64 0)
+			(hide yes)
+			(show_name no)
+			(do_not_autoplace no)
+			(effects
+				(font
+					(size 1.27 1.27)
+				)
+			)
+		)
+		(property "Supplier" "JLCPCB"
+			(at 38.1 40.64 0)
+			(hide yes)
+			(show_name no)
+			(do_not_autoplace no)
+			(effects
+				(font
+					(size 1.27 1.27)
+				)
+			)
+		)
 		(pin "1"
 		)
@@
 			(at 78.74 88.9 0)
 			(hide yes)
+			(show_name no)
+			(do_not_autoplace no)
+			(effects
+				(font
+					(size 1.27 1.27)
+				)
+			)
+		)
+		(property "LCSC" "C603786"
+			(at 78.74 88.9 0)
+			(hide yes)
+			(show_name no)
+			(do_not_autoplace no)
+			(effects
+				(font
+					(size 1.27 1.27)
+				)
+			)
+		)
+		(property "JLCPCB Manufacturer" "onsemi"
+			(at 78.74 88.9 0)
+			(hide yes)
+			(show_name no)
+			(do_not_autoplace no)
+			(effects
+				(font
+					(size 1.27 1.27)
+				)
+			)
+		)
+		(property "JLCPCB Part #" "NCP718ASN500T1G"
+			(at 78.74 88.9 0)
+			(hide yes)
