File: kicad/the_harp/Controls and LEDs.kicad_sch (KiCad schematic)
At the start: 45 parts, among them SW101 Snap/Glide, SW102 Bypass mode, SW103 Exp target

Commit message: Face as The Alchemist's: four knobs, three ON-ON-ON toggles
The Relic's six knobs and three toggles did not fit the four jacks: the
outer lower-row pots' pins sat on the upper jacks' rear pads and the outer
toggles over the jack bodies.

- Knobs: Mix, Sustain, Strings (row +38), Jawari (0, +13); RV104/RV106
  removed. Pots on PA0, PA1, PA2, PA4.
- Toggles: Taiway 100-DP6-T200B1M2QE ON-ON-ON (The Alchemist's part),
  Tuning Follow/Key/Drone and Brightness Dark/Warm/Glassy at (+-20, +13),
  Retune Snap/Glide/Lock at (0, -5); two MCU inputs each (PE11-PE15, PB10).
- PCB: toggles on the Alchemist footprint, RV104/RV106 deleted, bypass
  footswitch on R2816 pads, R405/D402 moved off J403's rear pads. No
  through-hole pad over a jack.
- Docs and design report: decision 13, face schedule, pin map, firmware
  requirements (TUN-11 Lock, TGL-1..3, bypass mode and expression target in
  the secondary layer).

Co-Authored-By: Claude Opus 5.5 <noreply@anthropic.com>
Claude-Session: https://claude.ai/code/session_01ToUUHuo6mg178NkLtQkDLg
Parts:
- removed C104, C106: 100n, Capacitor_SMD:C_0603_1608Metric, symbol Device:C
- removed R104, R106: 1k, Resistor_SMD:R_0603_1608Metric, symbol Device:R
- removed RV104, RV106: B10K, Potentiometer_THT:RD901F4015R1B10K00DL1, symbol POT:RD901F-40-15R1-B10K-00DL1
- added unit 2 of SW101
- added unit 2 of SW102
- added unit 2 of SW103
- SW101: value Snap/Glide -> 100-DP6; footprint SPDT Switches:SPDT love my Switches -> SPDT Switches:100DP3T1B2M2QE; symbol Switch:SW_SPDT -> Switch:SW_DPDT_x2; Manufacturer (none) -> Taiway; Mfg Part # (none) -> 100-DP6-T200B1M2QE; Supplier (none) -> LMS; now not fitted
- SW102: value Bypass mode -> 100-DP6; footprint SPDT Switches:SPDT love my Switches -> SPDT Switches:100DP3T1B2M2QE; symbol Switch:SW_SPDT -> Switch:SW_DPDT_x2; Manufacturer (none) -> Taiway; Mfg Part # (none) -> 100-DP6-T200B1M2QE; Supplier (none) -> LMS; now not fitted
- SW103: value Exp target -> 100-DP6; footprint SPDT Switches:SPDT love my Switches -> SPDT Switches:100DP3T1B2M2QE; symbol Switch:SW_SPDT -> Switch:SW_DPDT_x2; Manufacturer (none) -> Taiway; Mfg Part # (none) -> 100-DP6-T200B1M2QE; Supplier (none) -> LMS; now not fitted
Connections:
- net GND: now also SW101.5 (B), SW102.5 (B), SW103.5 (B)
- net TOG1_A: now reaches SW101.3 (C)
- net TOG2_A: now reaches SW102.3 (C)
- net TOG3_A: now reaches SW103.3 (C)
- net TOG1: no longer names the net of SW101.1 (A)
- net TOG2: no longer names the net of SW102.1 (A)
- net TOG3: no longer names the net of SW103.1 (A)
- new net TOG1_B: SW101.4 (A)
- new net TOG2_B: SW102.4 (A)
- new net TOG3_B: SW103.4 (A)
- no-connect marks 3 -> 6
Other:
- note added: "Controls and LEDs. Four B10K pots on the Alchemist grid: Mix, Sustain, Strings (row +38) and Jawari (0, +13), across +3V3, wipers to ADC1 PA0, PA1, PA2, PA4 through 1k / 100n. Three Taiway 100-DP6 ON-ON-ON toggles, as The Alchemist: Tuning (-20, +13), Brightness (+20, +13), Retune (0, -5). Commons (2, 5) to GND, pins 3 and 4 to two MCU inputs with internal pull-ups: up = A low B high, centre = bo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"
- note removed: "Controls and LEDs. Six B10K pots on the Relic/Alchemist grid (rows +38 / +13, columns -20 / 0 / +20) across +3V3, wipers to ADC1 PA0-PA5 through 1k / 100n. Three SPDT toggles (row -5) pull PE12-PE14 to ground; internal pull-ups. Twelve 0603 note LEDs, C to B, on PD0-PD11 (one port write), 1k each, behind 3 mm light pipes at face Y -18."
- moved on the sheet: C105, D101, D102, D103, D104, D105, D106, D107, D108, D109, D110, D111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
