File: kicad/the_harp/MCU.kicad_sch (KiCad schematic)
At the start: 23 parts, among them U201 STM32H750VBT6, U202 W25Q128JVSIQ, Y201 25MHz 9pF

Commit message: Face as The Alchemist's: four knobs, three ON-ON-ON toggles
The Relic's six knobs and three toggles did not fit the four jacks: the
outer lower-row pots' pins sat on the upper jacks' rear pads and the outer
toggles over the jack bodies.

- Knobs: Mix, Sustain, Strings (row +38), Jawari (0, +13); RV104/RV106
  removed. Pots on PA0, PA1, PA2, PA4.
- Toggles: Taiway 100-DP6-T200B1M2QE ON-ON-ON (The Alchemist's part),
  Tuning Follow/Key/Drone and Brightness Dark/Warm/Glassy at (+-20, +13),
  Retune Snap/Glide/Lock at (0, -5); two MCU inputs each (PE11-PE15, PB10).
- PCB: toggles on the Alchemist footprint, RV104/RV106 deleted, bypass
  footswitch on R2816 pads, R405/D402 moved off J403's rear pads. No
  through-hole pad over a jack.
- Docs and design report: decision 13, face schedule, pin map, firmware
  requirements (TUN-11 Lock, TGL-1..3, bypass mode and expression target in
  the secondary layer).

Co-Authored-By: Claude Opus 5.5 <noreply@anthropic.com>
Claude-Session: https://claude.ai/code/session_01ToUUHuo6mg178NkLtQkDLg
Connections:
- net TOG1_A: now reaches U201.41 (PE11)
- net TOG3_A: now reaches U201.45 (PE15)
- net TOG3_B: now reaches U201.46 (PB10)
- net POT4: no longer names the net of U201.25 (PA3)
- net POT6: no longer names the net of U201.29 (PA5)
- net TOG1 renamed TOG1_B
- net TOG2 renamed TOG2_A
- net TOG3 renamed TOG2_B
- no-connect marks 35 -> 34
