File: kicad/the_harp/The Harp.kicad_pcb (KiCad board)
At the start: 4 copper layers, 56 x 94.5 mm, 26 parts, among them J401 PJ-063AH, J402 NMJ6HCD2, J403 NMJ6HCD2, J404 NMJ6HCD2, J405 Bypass FSW, J406 NMJ6HCD2, K401 G6K-2F-Y, Q401 2N7002, Q402 2N7002, SW101 100-DP6, SW102 100-DP6, SW103 100-DP6

Commit message: pulled pcb
Parts:
- added C101: 100n, Capacitor_SMD:C_0603_1608Metric, F.Cu at (261.1, 98.3)
- added C102: 100n, Capacitor_SMD:C_0603_1608Metric, F.Cu at (261.1, 100.8)
- added C103: 100n, Capacitor_SMD:C_0603_1608Metric, F.Cu at (261.1, 103.3)
- added C105: 100n, Capacitor_SMD:C_0603_1608Metric, F.Cu at (261.1, 105.8)
- added C201: 2.2u, Capacitor_SMD:C_0603_1608Metric, F.Cu at (229.0, 98.3)
- added C202: 2.2u, Capacitor_SMD:C_0603_1608Metric, F.Cu at (229.0, 100.8)
- added C203: 4.7u, Capacitor_SMD:C_0805_2012Metric, F.Cu at (210.7, 117.0)
- added C204: 100n, Capacitor_SMD:C_0603_1608Metric, F.Cu at (229.0, 103.3)
- added C205: 100n, Capacitor_SMD:C_0603_1608Metric, F.Cu at (229.0, 105.8)
- added C206: 100n, Capacitor_SMD:C_0603_1608Metric, F.Cu at (229.0, 108.3)
- added C207: 100n, Capacitor_SMD:C_0603_1608Metric, F.Cu at (229.0, 110.8)
- added C208: 100n, Capacitor_SMD:C_0603_1608Metric, F.Cu at (229.0, 113.3)
- added C209: 1u, Capacitor_SMD:C_0603_1608Metric, F.Cu at (233.0, 98.3)
- added C210: 100n, Capacitor_SMD:C_0603_1608Metric, F.Cu at (233.0, 100.8)
- added C211: 8p, Capacitor_SMD:C_0603_1608Metric, F.Cu at (233.0, 103.3)
- added C212: 8p, Capacitor_SMD:C_0603_1608Metric, F.Cu at (233.0, 105.8)
- added C213: 100n, Capacitor_SMD:C_0603_1608Metric, F.Cu at (233.0, 108.3)
- added C214: 100n, Capacitor_SMD:C_0603_1608Metric, F.Cu at (233.0, 110.8)
- added C301: 2.2u, Capacitor_SMD:C_0603_1608Metric, F.Cu at (216.2, 127.5)
- added C302: 2.2u, Capacitor_SMD:C_0603_1608Metric, F.Cu at (216.2, 130.0)
- added C303: 10u, Capacitor_SMD:C_1206_3216Metric, F.Cu at (211.3, 140.7)
- added C304: 100n, Capacitor_SMD:C_0603_1608Metric, F.Cu at (216.2, 132.5)
- added C305: 100n, Capacitor_SMD:C_0603_1608Metric, F.Cu at (216.2, 135.0)
- added C306: 22u, Capacitor_SMD:C_1210_3225Metric, F.Cu at (211.3, 128.4)
- added C307: 22u, Capacitor_SMD:C_1210_3225Metric, F.Cu at (211.3, 132.6)
- added C308: 47u, Capacitor_SMD:C_1210_3225Metric, F.Cu at (211.3, 136.9)
- added C309: 2.2u, Capacitor_SMD:C_0603_1608Metric, F.Cu at (216.2, 137.5)
- added C310: 2.2u, Capacitor_SMD:C_0603_1608Metric, F.Cu at (220.2, 127.5)
- added C311: 2.2u, Capacitor_SMD:C_0603_1608Metric, F.Cu at (220.2, 130.0)
- added C312: 2.2u, Capacitor_SMD:C_0603_1608Metric, F.Cu at (220.2, 132.5)
- added C409: 100n, Capacitor_SMD:C_0603_1608Metric, F.Cu at (258.5, 127.5)
- added C410: 100n, Capacitor_SMD:C_0603_1608Metric, F.Cu at (258.5, 130.0)
- added C411: 100n, Capacitor_SMD:C_0603_1608Metric, F.Cu at (258.5, 132.5)
- added C412: 2.7n, Capacitor_SMD:C_0603_1608Metric, F.Cu at (258.5, 135.0)
- added C501: 100n, Capacitor_SMD:C_0603_1608Metric, F.Cu at (243.1, 144.6)
- added C502: 10u, Capacitor_SMD:CP_Elec_4x5.8, F.Cu at (237.2, 146.2)
- added C503: 100n, Capacitor_SMD:C_0603_1608Metric, F.Cu at (243.1, 147.1)
- added C504: 100n, Capacitor_SMD:C_0603_1608Metric, F.Cu at (243.1, 149.6)
- added C505: 100n, Capacitor_SMD:C_0603_1608Metric, F.Cu at (243.1, 152.1)
- added C506: 100n, Capacitor_SMD:C_0603_1608Metric, F.Cu at (247.1, 144.6)
- added C507: 100n, Capacitor_SMD:C_0603_1608Metric, F.Cu at (247.1, 147.1)
- added C508: 10u, Capacitor_SMD:CP_Elec_4x5.8, F.Cu at (237.2, 152.1)
- added C509: 100n, Capacitor_SMD:C_0603_1608Metric, F.Cu at (247.1, 149.6)
- added C601: 100p, Capacitor_SMD:C_0603_1608Metric, F.Cu at (235.3, 127.5)
- added C602: 100p, Capacitor_SMD:C_0603_1608Metric, F.Cu at (235.3, 130.0)
- added C603: 1n, Capacitor_SMD:C_0603_1608Metric, F.Cu at (235.3, 132.5)
- added C604: 1n, Capacitor_SMD:C_0603_1608Metric, F.Cu at (235.3, 135.0)
- added C605: 2.7n, Capacitor_SMD:C_0603_1608Metric, F.Cu at (235.3, 137.5)
- added C606: 100p, Capacitor_SMD:C_0603_1608Metric, F.Cu at (235.3, 140.1)
- added C607: 100p, Capacitor_SMD:C_0603_1608Metric, F.Cu at (239.3, 127.5)
- added C608: 100n, Capacitor_SMD:C_0603_1608Metric, F.Cu at (239.3, 130.0)
- added C609: 100n, Capacitor_SMD:C_0603_1608Metric, F.Cu at (239.3, 132.5)
- added C610: 100n, Capacitor_SMD:C_0603_1608Metric, F.Cu at (239.3, 135.0)
- added C701: 100n, Capacitor_SMD:C_1206_3216Metric, F.Cu at (252.3, 117.5)
- added C702: 220p, Capacitor_SMD:C_0603_1608Metric, F.Cu at (243.0, 98.3)
- added C703: 100n, Capacitor_SMD:C_0603_1608Metric, F.Cu at (243.0, 100.8)
- added C704: 10u, Capacitor_Tantalum_SMD:CP_EIA-3216-12_Kemet-S, F.Cu at (252.4, 111.1)
- added C705: 10u, Capacitor_Tantalum_SMD:CP_EIA-3216-12_Kemet-S, F.Cu at (252.4, 114.3)
- added C706: 100n, Capacitor_SMD:C_0603_1608Metric, F.Cu at (243.0, 103.3)
- added C707: 10u, Capacitor_SMD:C_0805_2012Metric, F.Cu at (251.7, 120.7)
- added D101: LED, LED_SMD:LED_0603_1608Metric, F.Cu at (261.1, 110.8)
- added D102: LED, LED_SMD:LED_0603_1608Metric, F.Cu at (261.1, 113.4)
- added D103: LED, LED_SMD:LED_0603_1608Metric, F.Cu at (261.1, 116.0)
- added D104: LED, LED_SMD:LED_0603_1608Metric, F.Cu at (261.1, 118.6)
- added D105: LED, LED_SMD:LED_0603_1608Metric, F.Cu at (265.2, 110.8)
- added D106: LED, LED_SMD:LED_0603_1608Metric, F.Cu at (265.2, 113.4)
- added D107: LED, LED_SMD:LED_0603_1608Metric, F.Cu at (265.2, 116.0)
- added D108: LED, LED_SMD:LED_0603_1608Metric, F.Cu at (265.2, 118.6)
- added D109: LED, LED_SMD:LED_0603_1608Metric, F.Cu at (269.2, 110.8)
- added D110: LED, LED_SMD:LED_0603_1608Metric, F.Cu at (269.2, 113.4)
- added D111: LED, LED_SMD:LED_0603_1608Metric, F.Cu at (269.2, 116.0)
- added D112: LED, LED_SMD:LED_0603_1608Metric, F.Cu at (269.2, 118.6)
- added D114: RED_LED, LED_THT:LED_D3.0mm, F.Cu at (270.2, 135.0)
- added D301: SMAJ10CA, Diode_SMD:D_SMA, F.Cu at (218.2, 141.1)
- added D302: PMEG3010ER, Diode_SMD:Nexperia_CFP3_SOD-123W, F.Cu at (211.3, 144.0)
- added D403: PESD5V0U1BB,115, Diode_SMD:D_SOD-523, F.Cu at (266.7, 133.5)
- added D404: PESD5V0U1BB,115, Diode_SMD:D_SOD-523, F.Cu at (266.7, 135.9)
- added D405: PESD5V0U1BB,115, Diode_SMD:D_SOD-523, F.Cu at (266.7, 138.4)
- added D406: PESD5V0U1BB,115, Diode_SMD:D_SOD-523, F.Cu at (266.7, 140.8)
- added FB201: 220R, Inductor_SMD:L_0603_1608Metric, F.Cu at (233.0, 113.3)
- added FB301: 600R, Inductor_SMD:L_0603_1608Metric, F.Cu at (220.2, 135.0)
- added FB302: 600R, Inductor_SMD:L_0603_1608Metric, F.Cu at (220.2, 137.5)
- added FB303: 600R, Inductor_SMD:L_0603_1608Metric, F.Cu at (224.2, 127.5)
- added J407: Hold FSW, Resistor_SMD:R_2816_7142Metric_Pad3.20x4.45mm_HandSolder, F.Cu at (269.9, 129.3)
- added L301: 10u, Inductor_SMD:L_APV_ANR5020, F.Cu at (225.6, 142.1)
- added Q403: 2N7002, Package_TO_SOT_SMD:SOT-23, F.Cu at (270.9, 144.6)
- added R101: 1k, Resistor_SMD:R_0603_1608Metric, F.Cu at (261.1, 108.3)
- added R102: 1k, Resistor_SMD:R_0603_1608Metric, F.Cu at (265.1, 98.3)
- added R103: 1k, Resistor_SMD:R_0603_1608Metric, F.Cu at (265.1, 100.8)
- added R105: 1k, Resistor_SMD:R_0603_1608Metric, F.Cu at (265.1, 103.3)
- added R107: 1k, Resistor_SMD:R_0603_1608Metric, F.Cu at (265.1, 105.8)
- added R108: 1k, Resistor_SMD:R_0603_1608Metric, F.Cu at (265.1, 108.3)
- added R109: 1k, Resistor_SMD:R_0603_1608Metric, F.Cu at (269.1, 98.3)
- added R110: 1k, Resistor_SMD:R_0603_1608Metric, F.Cu at (269.1, 100.8)
- added R111: 1k, Resistor_SMD:R_0603_1608Metric, F.Cu at (269.1, 103.3)
- added R112: 1k, Resistor_SMD:R_0603_1608Metric, F.Cu at (269.1, 105.8)
- added R113: 1k, Resistor_SMD:R_0603_1608Metric, F.Cu at (269.1, 108.3)
- added R114: 1k, Resistor_SMD:R_0603_1608Metric, F.Cu at (273.1, 98.3)
- added R115: 1k, Resistor_SMD:R_0603_1608Metric, F.Cu at (273.1, 100.8)
- added R116: 1k, Resistor_SMD:R_0603_1608Metric, F.Cu at (273.1, 103.3)
- added R117: 1k, Resistor_SMD:R_0603_1608Metric, F.Cu at (273.1, 105.8)
- added R118: 1k, Resistor_SMD:R_0603_1608Metric, F.Cu at (273.1, 108.3)
- added R201: 10k, Resistor_SMD:R_0603_1608Metric, F.Cu at (237.0, 98.3)
- added R202: 22R, Resistor_SMD:R_0603_1608Metric, F.Cu at (237.0, 100.8)
- added R203: 22R, Resistor_SMD:R_0603_1608Metric, F.Cu at (237.0, 103.3)
- added R204: 10k, Resistor_SMD:R_0603_1608Metric, F.Cu at (237.0, 105.8)
- added R301: 49.9, Resistor_SMD:R_0603_1608Metric, F.Cu at (224.2, 130.0)
- added R302: 100k, Resistor_SMD:R_0603_1608Metric, F.Cu at (224.2, 132.5)
- added R303: 22k, Resistor_SMD:R_0603_1608Metric, F.Cu at (224.2, 135.0)
- added R411: 1k, Resistor_SMD:R_0805_2012Metric, F.Cu at (262.7, 127.7)
- added R412: 100R, Resistor_SMD:R_0805_2012Metric, F.Cu at (262.7, 130.7)
- added R413: 100k, Resistor_SMD:R_0805_2012Metric, F.Cu at (262.7, 133.6)
- added R414: 1k, Resistor_SMD:R_0805_2012Metric, F.Cu at (262.7, 136.6)
- added R415: 100R, Resistor_SMD:R_0603_1608Metric, F.Cu at (258.5, 137.5)
- added R416: 1k, Resistor_SMD:R_0603_1608Metric, F.Cu at (258.5, 140.1)
- added R417: 100k, Resistor_SMD:R_0603_1608Metric, F.Cu at (258.5, 142.6)
- added R418: 100R, Resistor_SMD:R_0603_1608Metric, F.Cu at (258.5, 145.1)
- added R501: 5k1, Resistor_SMD:R_0603_1608Metric, F.Cu at (247.1, 152.1)
- added R502: 1k, Resistor_SMD:R_0603_1608Metric, F.Cu at (251.1, 144.6)
- added R503: 1k, Resistor_SMD:R_0603_1608Metric, F.Cu at (251.1, 147.1)
- added R504: 10R, Resistor_SMD:R_0603_1608Metric, F.Cu at (251.1, 149.6)
- added R505: 10R, Resistor_SMD:R_0603_1608Metric, F.Cu at (251.1, 152.1)
- added R601: 1k, Resistor_SMD:R_0603_1608Metric, F.Cu at (239.3, 137.5)
- added R602: 1.05k, Resistor_SMD:R_0603_1608Metric, F.Cu at (239.3, 140.1)
- added R603: 620, Resistor_SMD:R_0603_1608Metric, F.Cu at (243.4, 127.5)
- added R604: 620, Resistor_SMD:R_0603_1608Metric, F.Cu at (243.4, 130.0)
- added R605: 40.2, Resistor_SMD:R_0603_1608Metric, F.Cu at (243.4, 132.5)
- added R606: 40.2, Resistor_SMD:R_0603_1608Metric, F.Cu at (243.4, 135.0)
- added R701: 1M, Resistor_SMD:R_0603_1608Metric, F.Cu at (243.0, 105.8)
- added R702: 1M, Resistor_SMD:R_0603_1608Metric, F.Cu at (243.0, 108.3)
- added R703: 0R, Resistor_SMD:R_0603_1608Metric, F.Cu at (247.1, 98.3)
- added R704: 0R, Resistor_SMD:R_0603_1608Metric, F.Cu at (247.1, 100.8)
- added R705: 49.9, Resistor_SMD:R_0603_1608Metric, F.Cu at (247.1, 103.3)
- added R706: 10k, Resistor_SMD:R_0603_1608Metric, F.Cu at (247.1, 105.8)
- added R707: 10k, Resistor_SMD:R_0603_1608Metric, F.Cu at (247.1, 108.3)
- added R708: 10k, Resistor_SMD:R_0603_1608Metric, F.Cu at (251.1, 98.3)
- added R709: 10k, Resistor_SMD:R_0603_1608Metric, F.Cu at (251.1, 100.8)
- added R710: 100R, Resistor_SMD:R_0603_1608Metric, F.Cu at (251.1, 103.3)
- added R711: 1M, Resistor_SMD:R_0603_1608Metric, F.Cu at (251.1, 105.8)
- added R714: 10k, Resistor_SMD:R_0603_1608Metric, F.Cu at (251.1, 108.3)
- added R715: 10k, Resistor_SMD:R_0603_1608Metric, F.Cu at (255.1, 98.3)
- added R716: 10k, Resistor_SMD:R_0603_1608Metric, F.Cu at (255.1, 100.8)
- added R717: 10k, Resistor_SMD:R_0603_1608Metric, F.Cu at (255.1, 103.3)
- added R718: 100R, Resistor_SMD:R_0603_1608Metric, F.Cu at (255.1, 105.8)
- added R719: 1M, Resistor_SMD:R_0603_1608Metric, F.Cu at (255.1, 108.3)
- added U201: STM32H750VBT6, Package_QFP:LQFP-100_14x14mm_P0.5mm, F.Cu at (217.8, 106.3)
- added U301: TPS54202DDC, Package_TO_SOT_SMD:SOT-23-6, F.Cu at (228.8, 128.7)
- added U302: NCP718ASN500T1G, Package_TO_SOT_SMD:TSOT-23-5, F.Cu at (228.8, 133.3)
- added U401: MCP6001T-I/OT, Package_TO_SOT_SMD:SOT-23-5, F.Cu at (271.1, 140.1)
- added U501: OPA2348AIDR, Package_SO:SOIC-8_3.9x4.9mm_P1.27mm, F.Cu at (245.3, 156.7)
- added U601: THS4522IPW, Package_SO:TSSOP-16_4.4x5mm_P0.65mm, F.Cu at (250.1, 129.5)
- added U701: OPA2365AIDR, Package_SO:SOIC-8_3.9x4.9mm_P1.27mm, F.Cu at (245.3, 112.9)
- added U702: OPA1688IDR, Package_SO:SOIC-8_3.9x4.9mm_P1.27mm, F.Cu at (245.3, 119.5)
- added W201: SWD needle, LIB_STLINK:SEGGER_8.06.05_6-PIN_NEEDLE_ADAPTER, F.Cu at (234.0, 119.2)
- added Y201: 25MHz 9pF, Crystal:Crystal_SMD_2016-4Pin_2.0x1.6mm, F.Cu at (210.5, 120.3)
Connections:
- C408 pad 1: (no net) -> FSW_BYPASS_IN
- C408 pad 2: (no net) -> GND
- D113 pad 1: (no net) -> /Jacks and Bypass/LED_EFF_K
- D113 pad 2: (no net) -> +9V
- D402 pad 1: (no net) -> /Jacks and Bypass/RELAY_COIL
- D402 pad 2: (no net) -> /Jacks and Bypass/RELAY_LOW
- J401 pad 1: (no net) -> GND
- J401 pad 2: (no net) -> /Power/DC_IN
- J402 pad R: (no net) -> GND
- J402 pad RN: (no net) -> unconnected-(J402-PadRN)
- J402 pad S: (no net) -> GND
- J402 pad SN: (no net) -> unconnected-(J402-PadSN)
- J402 pad T: (no net) -> /Jacks and Bypass/IN
- J402 pad TN: (no net) -> unconnected-(J402-PadTN)
- J403 pad R: (no net) -> unconnected-(J403-PadR)
- J403 pad RN: (no net) -> unconnected-(J403-PadRN)
- J403 pad S: (no net) -> GND
- J403 pad SN: (no net) -> unconnected-(J403-PadSN)
- J403 pad T: (no net) -> /Jacks and Bypass/OUT_L
- J403 pad TN: (no net) -> unconnected-(J403-PadTN)
- J404 pad R: (no net) -> unconnected-(J404-PadR)
- J404 pad RN: (no net) -> unconnected-(J404-PadRN)
- J404 pad S: (no net) -> GND
- J404 pad SN: (no net) -> unconnected-(J404-PadSN)
- J404 pad T: (no net) -> EFFECT_OUT_R
- J404 pad TN: (no net) -> unconnected-(J404-PadTN)
- J405 pad 1: (no net) -> /Jacks and Bypass/FSW_BYPASS
- J405 pad 2: (no net) -> GND
- J406 pad R: (no net) -> /Jacks and Bypass/EXP_RING
- J406 pad RN: (no net) -> unconnected-(J406-PadRN)
- J406 pad S: (no net) -> GND
- J406 pad SN: (no net) -> unconnected-(J406-PadSN)
- J406 pad T: (no net) -> /Jacks and Bypass/EXP_TIP
- J406 pad TN: (no net) -> unconnected-(J406-PadTN)
- K401 pad 1: (no net) -> /Jacks and Bypass/RELAY_COIL
- K401 pad 2: (no net) -> /Jacks and Bypass/IN
- K401 pad 3: (no net) -> /Jacks and Bypass/OUT_L
- K401 pad 4: (no net) -> EFFECT_OUT_L
- K401 pad 5: (no net) -> /Jacks and Bypass/IN
- K401 pad 6: (no net) -> EFFECT_IN
- K401 pad 7: (no net) -> GND
- K401 pad 8: (no net) -> /Jacks and Bypass/RELAY_LOW
- Q401 pad 1: (no net) -> /Jacks and Bypass/RELAY_G
- Q401 pad 2: (no net) -> GND
- Q401 pad 3: (no net) -> /Jacks and Bypass/RELAY_LOW
- Q402 pad 1: (no net) -> /Jacks and Bypass/LED_EFF_G
- Q402 pad 2: (no net) -> GND
- Q402 pad 3: (no net) -> /Jacks and Bypass/LED_EFF_LOW
- R404 pad 1: (no net) -> /Jacks and Bypass/LED_EFF_K
- R404 pad 2: (no net) -> /Jacks and Bypass/LED_EFF_LOW
- R405 pad 1: (no net) -> +9V
- R405 pad 2: (no net) -> /Jacks and Bypass/RELAY_COIL
- R406 pad 1: (no net) -> RELAY_DRV
- R406 pad 2: (no net) -> /Jacks and Bypass/RELAY_G
- R407 pad 1: (no net) -> /Jacks and Bypass/RELAY_G
- R407 pad 2: (no net) -> GND
- R408 pad 1: (no net) -> LED_EFFECT_DRV
- R408 pad 2: (no net) -> /Jacks and Bypass/LED_EFF_G
- R409 pad 1: (no net) -> /Jacks and Bypass/LED_EFF_G
- R409 pad 2: (no net) -> GND
- R410 pad 1: (no net) -> /Jacks and Bypass/FSW_BYPASS
- R410 pad 2: (no net) -> FSW_BYPASS_IN
- RV101 pad 1: (no net) -> GND
- RV101 pad 2: (no net) -> /Controls and LEDs/POT1_W
- RV101 pad 3: (no net) -> +3V3
- RV101 pad MH1: (no net) -> GND
- RV101 pad MH2: (no net) -> GND
- RV102 pad 1: (no net) -> GND
- RV102 pad 2: (no net) -> /Controls and LEDs/POT2_W
- RV102 pad 3: (no net) -> +3V3
- RV102 pad MH1: (no net) -> GND
- RV102 pad MH2: (no net) -> GND
- RV103 pad 1: (no net) -> GND
- RV103 pad 2: (no net) -> /Controls and LEDs/POT3_W
- RV103 pad 3: (no net) -> +3V3
- RV103 pad MH1: (no net) -> GND
- RV103 pad MH2: (no net) -> GND
- RV105 pad 1: (no net) -> GND
- RV105 pad 2: (no net) -> /Controls and LEDs/POT5_W
- RV105 pad 3: (no net) -> +3V3
- RV105 pad MH1: (no net) -> GND
- RV105 pad MH2: (no net) -> GND
- SW101 pad 1: (no net) -> unconnected-(SW101A-A-Pad1)
- SW101 pad 2: (no net) -> GND
- SW101 pad 3: (no net) -> TOG1_A
- SW101 pad 4: (no net) -> TOG1_B
- SW101 pad 5: (no net) -> GND
- SW101 pad 6: (no net) -> unconnected-(SW101B-C-Pad6)
- SW102 pad 1: (no net) -> unconnected-(SW102A-A-Pad1)
- SW102 pad 2: (no net) -> GND
- SW102 pad 3: (no net) -> TOG2_A
- SW102 pad 4: (no net) -> TOG2_B
- SW102 pad 5: (no net) -> GND
- SW102 pad 6: (no net) -> unconnected-(SW102B-C-Pad6)
- SW103 pad 1: (no net) -> unconnected-(SW103A-A-Pad1)
- SW103 pad 2: (no net) -> GND
- SW103 pad 3: (no net) -> TOG3_A
- SW103 pad 4: (no net) -> TOG3_B
- SW103 pad 5: (no net) -> GND
- SW103 pad 6: (no net) -> unconnected-(SW103B-C-Pad6)
