File: kicad/the_harp/The Harp.kicad_pcb (KiCad board)
At the start: 4 copper layers, 56 x 94.5 mm, 181 parts, among them IC501 AK4621EF, J401 PJ-063AH, J402 NMJ6HCD2, J403 NMJ6HCD2, J404 NMJ6HCD2, J405 Bypass FSW, J406 NMJ6HCD2, J407 Hold FSW, J408 OLED 0.91 128x32, K401 G6K-2F-Y, Q401 2N7002, Q402 2N7002, Q403 2N7002, SW101 100-DP6, SW102 100-DP6, SW103 100-DP6, U201 STM32H750VBT6, U202 W25Q128JVSIQ, U301 TPS54202DDC, U302 NCP718ASN500T1G, U401 MCP6001T-I/OT, U501 OPA2348AIDR, U601 THS4522IPW, U701 OPA2365AIDR, U702 OPA1688IDR, Y201 25MHz 9pF

Commit message: Revert In2 pours: the rails go back to tracks
Reverts PR #15. The block-style pours were not manufacturable. The board is
as before it: +3V3 / +5V / +9V as 0.5 / 0.6 mm tracks on In2.Cu, 1546 tracks,
302 vias, 32 connections open. The pour scripts and the docs on them are
removed with it.

Co-Authored-By: Claude Sonnet 5.5 <noreply@anthropic.com>
Claude-Session: https://claude.ai/code/session_016hDejPHPgG8auBLMyByYZK
Routing:
- net +3V3: track 37.3 -> 310.7 mm
- net +9V: track 6.16 -> 238.1 mm
- net +5V: track 22.2 -> 198.6 mm
- removed copper zone on In2.Cu, net +3V3
- removed copper zone on In2.Cu, net +5V
- removed copper zone on In2.Cu, net +9V
