File: kicad/the_harp/The Harp.kicad_pcb (KiCad board)
At the start: 4 copper layers, 56 x 94.5 mm, 181 parts, among them IC501 AK4621EF, J401 PJ-063AH, J402 NMJ6HCD2, J403 NMJ6HCD2, J404 NMJ6HCD2, J405 Bypass FSW, J406 NMJ6HCD2, J407 Hold FSW, J408 OLED 0.91 128x32, K401 G6K-2F-Y, Q401 2N7002, Q402 2N7002, Q403 2N7002, SW101 100-DP6, SW102 100-DP6, SW103 100-DP6, U201 STM32H750VBT6, U202 W25Q128JVSIQ, U301 TPS54202DDC, U302 NCP718ASN500T1G, U401 MCP6001T-I/OT, U501 OPA2348AIDR, U601 THS4522IPW, U701 OPA2365AIDR, U702 OPA1688IDR, Y201 25MHz 9pF

Commit message: update
Parts:
- removed C101, C102, C103, C104, C105, C204, C205, C206, C207, C208, C210, C214, C304, C305, C408, C409, C410, C411, C501, C503, C509, C608, C609, C610, C618, C703, C706: 100n, Capacitor_SMD:C_0603_1608Metric
- removed C201, C202, C301, C302, C309, C310, C311, C312: 2.2u, Capacitor_SMD:C_0603_1608Metric
- removed C203: 4.7u, Capacitor_SMD:C_0805_2012Metric
- removed C209: 1u, Capacitor_SMD:C_0603_1608Metric
- removed C211, C212: 8p, Capacitor_SMD:C_0603_1608Metric
- removed C303: 10u, Capacitor_SMD:C_1206_3216Metric
- removed C306, C307: 22u, Capacitor_SMD:C_1210_3225Metric
- removed C308: 47u, Capacitor_SMD:C_1210_3225Metric
- removed C412, C605, C615: 2.7n, Capacitor_SMD:C_0603_1608Metric
- removed C502: 10u, Capacitor_SMD:CP_Elec_4x5.8
- removed C601, C602, C606, C607, C611, C612, C616, C617: 100p, Capacitor_SMD:C_0603_1608Metric
- removed C603, C604, C613, C614: 1n, Capacitor_SMD:C_0603_1608Metric
- removed C701, C708: 100n, Capacitor_SMD:C_1206_3216Metric
- removed C702, C709: 220p, Capacitor_SMD:C_0603_1608Metric
- removed C704, C705: 10u, Capacitor_Tantalum_SMD:CP_EIA-3216-12_Kemet-S
- removed C707: 10u, Capacitor_SMD:C_0805_2012Metric
- removed D114: RED_LED, LED_THT:LED_D3.0mm
- removed D301: SMAJ10CA, Diode_SMD:D_SMA
- removed D302: PMEG3010ER, Diode_SMD:Nexperia_CFP3_SOD-123W
- removed D402: 1N4148W, Diode_SMD:D_SOD-123
- removed D404, D405, D406: PESD5V0U1BB,115, Diode_SMD:D_SOD-523
- removed FB201: 220R, Inductor_SMD:L_0603_1608Metric
- removed FB301, FB302, FB303: 600R, Inductor_SMD:L_0603_1608Metric
- removed J403, J404, J406: NMJ6HCD2, Connector_Audio:Jack_6.35mm_Neutrik_NMJ6HCD2_Horizontal
- removed J405: Bypass FSW, Resistor_SMD:R_2816_7142Metric_Pad3.20x4.45mm_HandSolder
- removed J407: Hold FSW, Resistor_SMD:R_2816_7142Metric_Pad3.20x4.45mm_HandSolder
- removed J408: OLED 0.91 128x32, Connector_JST:JST_SH_SM04B-SRSS-TB_1x04-1MP_P1.00mm_Horizontal
- removed K401: G6K-2F-Y, Relay_SMD:Relay_DPDT_Omron_G6K-2F-Y
- removed L301: 10u, Inductor_SMD:L_APV_ANR5020
- removed Q401, Q402, Q403: 2N7002, Package_TO_SOT_SMD:SOT-23
- removed R101, R102, R103, R105, R416, R601, R607: 1k, Resistor_SMD:R_0603_1608Metric
- removed R107, R108: 4.7k, Resistor_SMD:R_0603_1608Metric
- removed R201, R204, R706, R708, R709, R714, R715, R716, R717: 10k, Resistor_SMD:R_0603_1608Metric
- removed R202, R203: 22R, Resistor_SMD:R_0603_1608Metric
- removed R301, R705, R722: 49.9, Resistor_SMD:R_0603_1608Metric
- removed R302, R417: 100k, Resistor_SMD:R_0603_1608Metric
- removed R303: 22k, Resistor_SMD:R_0603_1608Metric
- removed R405: 150R, Resistor_SMD:R_1206_3216Metric
- removed R406, R408, R412: 100R, Resistor_SMD:R_0805_2012Metric
- removed R407, R409, R413: 100k, Resistor_SMD:R_0805_2012Metric
- removed R410, R411, R414: 1k, Resistor_SMD:R_0805_2012Metric
- removed R415, R418, R710, R718: 100R, Resistor_SMD:R_0603_1608Metric
- removed R501: 5k1, Resistor_SMD:R_0603_1608Metric
- removed R504, R505: 10R, Resistor_SMD:R_0603_1608Metric
- removed R602, R608: 1.05k, Resistor_SMD:R_0603_1608Metric
- removed R603, R604, R609, R610: 620, Resistor_SMD:R_0603_1608Metric
- removed R605, R606, R611, R612: 40.2, Resistor_SMD:R_0603_1608Metric
- removed R701, R702, R711, R719, R720, R721: 1M, Resistor_SMD:R_0603_1608Metric
- removed R703, R704: 0R, Resistor_SMD:R_0603_1608Metric
- removed RV101, RV102, RV103, RV105: B10K, Potentiometer_THT:RD901F4015R1B10K00DL1
- removed U201: STM32H750VBT6, Package_QFP:LQFP-100_14x14mm_P0.5mm
- removed U202: W25Q128JVSIQ, Package_SO:SOIC-8_5.23x5.23mm_P1.27mm
- removed U301: TPS54202DDC, Package_TO_SOT_SMD:SOT-23-6
- removed U302: NCP718ASN500T1G, Package_TO_SOT_SMD:TSOT-23-5
- removed U401: MCP6001T-I/OT, Package_TO_SOT_SMD:SOT-23-5
- removed U501: OPA2348AIDR, Package_SO:SOIC-8_3.9x4.9mm_P1.27mm
- removed U601: THS4522IPW, Package_SO:TSSOP-16_4.4x5mm_P0.65mm
- removed U701: OPA2365AIDR, Package_SO:SOIC-8_3.9x4.9mm_P1.27mm
- removed U702: OPA1688IDR, Package_SO:SOIC-8_3.9x4.9mm_P1.27mm
- removed W201: SWD needle, LIB_STLINK:SEGGER_8.06.05_6-PIN_NEEDLE_ADAPTER
- removed Y201: 25MHz 9pF, Crystal:Crystal_SMD_2016-4Pin_2.0x1.6mm
Connections:
- C213 pad 1: /MCU/NRST -> unconnected-(C213-Pad1)
- C213 pad 2: GND -> unconnected-(C213-Pad2)
- C504 pad 1: +3V3 -> unconnected-(C504-Pad1)
- C504 pad 2: GND -> unconnected-(C504-Pad2)
- C505 pad 1: +3V3 -> unconnected-(C505-Pad1)
- C505 pad 2: GND -> unconnected-(C505-Pad2)
- C506 pad 1: +3V3 -> unconnected-(C506-Pad1)
- C506 pad 2: GND -> unconnected-(C506-Pad2)
- C507 pad 1: +5V -> unconnected-(C507-Pad1)
- C507 pad 2: GND -> unconnected-(C507-Pad2)
- C508 pad 1: +5V -> unconnected-(C508-Pad1)
- C508 pad 2: GND -> unconnected-(C508-Pad2)
- D113 pad 1: /Jacks and Bypass/LED_EFF_K -> unconnected-(D113-K-Pad1)
- D113 pad 2: +9V -> unconnected-(D113-A-Pad2)
- D403 pad 1: GND -> unconnected-(D403-A1-Pad1)
- D403 pad 2: /Jacks and Bypass/IN -> unconnected-(D403-A2-Pad2)
- D407 pad 1: GND -> unconnected-(D407-A1-Pad1)
- D407 pad 2: IN_R -> unconnected-(D407-A2-Pad2)
- IC501 pad 1: /Codec/VCOM -> unconnected-(IC501-VCOM-Pad1)
- IC501 pad 10: CODEC_MCLK -> unconnected-(IC501-MCLK-Pad10)
- IC501 pad 11: CODEC_LRCK -> unconnected-(IC501-LRCK-Pad11)
- IC501 pad 12: CODEC_BICK -> unconnected-(IC501-BICK-Pad12)
- IC501 pad 13: CODEC_SDTO -> unconnected-(IC501-SDTO-Pad13)
- IC501 pad 14: CODEC_SDTI -> unconnected-(IC501-SDTI-Pad14)
- IC501 pad 17: CODEC_CDTI -> unconnected-(IC501-CDTI/CKS0-Pad17)
- IC501 pad 18: CODEC_CCLK -> unconnected-(IC501-CCLK/CKS1-Pad18)
- IC501 pad 19: CODEC_CSN -> unconnected-(IC501-CSN/DIF-Pad19)
- IC501 pad 2: ADC_R_P -> unconnected-(IC501-AINR+-Pad2)
- IC501 pad 20: GND -> unconnected-(IC501-DFS0-Pad20)
- IC501 pad 21: /Codec/PDN -> unconnected-(IC501-PDN-Pad21)
- IC501 pad 22: GND -> unconnected-(IC501-DEM0-Pad22)
- IC501 pad 23: GND -> unconnected-(IC501-SDFIL-Pad23)
- IC501 pad 24: +3V3 -> unconnected-(IC501-TVDD-Pad24)
- IC501 pad 25: +3V3 -> unconnected-(IC501-DVDD-Pad25)
- IC501 pad 26: GND -> unconnected-(IC501-VSS2-Pad26)
- IC501 pad 27: DAC_L_N -> unconnected-(IC501-AOUTL--Pad27)
- IC501 pad 28: DAC_L_P -> unconnected-(IC501-AOUTL+-Pad28)
- IC501 pad 29: DAC_R_N -> unconnected-(IC501-AOUTR--Pad29)
- IC501 pad 3: ADC_R_N -> unconnected-(IC501-AINR--Pad3)
- IC501 pad 30: DAC_R_P -> unconnected-(IC501-AOUTR+-Pad30)
- IC501 pad 4: ADC_L_P -> unconnected-(IC501-AINL+-Pad4)
- IC501 pad 5: ADC_L_N -> unconnected-(IC501-AINL--Pad5)
- IC501 pad 6: +5V -> unconnected-(IC501-VREF-Pad6)
- IC501 pad 7: GND -> unconnected-(IC501-VSS1-Pad7)
- IC501 pad 8: +5V -> unconnected-(IC501-AVDD-Pad8)
- IC501 pad 9: +3V3 -> unconnected-(IC501-P/S-Pad9)
- J402 pad R: IN_R -> unconnected-(J402-PadR)
- J402 pad S: GND -> unconnected-(J402-PadS)
- J402 pad T: /Jacks and Bypass/IN -> unconnected-(J402-PadT)
- R404 pad 1: /Jacks and Bypass/LED_EFF_K -> unconnected-(R404-Pad1)
- R404 pad 2: /Jacks and Bypass/LED_EFF_LOW -> unconnected-(R404-Pad2)
- R707 pad 1: /Analog In and Out/OUTL_P -> unconnected-(R707-Pad1)
- R707 pad 2: VCOM_B -> unconnected-(R707-Pad2)
Routing:
- net (no net): track 0.00 -> 2254.0 mm, vias 0 -> 151
- net +3V3: track 310.7 -> 0.00 mm, vias 34 -> 0
- net unconnected-(D113-A-Pad2): track 0.00 -> 238.1 mm, vias 0 -> 6
- net +9V: track 238.1 -> 0.00 mm, vias 6 -> 0
- net +5V: track 198.6 -> 0.00 mm, vias 19 -> 0
- net VCOM_B: track 192.7 -> 0.00 mm, vias 7 -> 0
- net unconnected-(R707-Pad2): track 0.00 -> 192.7 mm, vias 0 -> 7
- net /Jacks and Bypass/IN: track 103.9 -> 0.00 mm, vias 1 -> 0
- net unconnected-(IC501-VCOM-Pad1): track 0.00 -> 85.5 mm, vias 0 -> 2
- net /Codec/VCOM: track 85.5 -> 0.00 mm, vias 2 -> 0
- net VCOM_A: track 75.9 -> 0.00 mm, vias 2 -> 0
- net EFFECT_OUT_L: track 73.4 -> 0.00 mm, vias 1 -> 0
- net EFFECT_IN: track 66.3 -> 0.00 mm, vias 1 -> 0
- net EXP: track 62.7 -> 0.00 mm, vias 3 -> 0
- net ADC_L_P: track 62.6 -> 0.00 mm, vias 4 -> 0
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- added copper zone on In1.Cu, net unconnected-(J402-PadS)
- removed copper zone on In1.Cu, net GND
