File: kicad/the_harp/The Harp.kicad_pcb (KiCad board)
At the start: 4 copper layers, 56 x 94.5 mm, 181 parts, among them IC501 AK4621EF, J401 PJ-063AH, J402 NMJ6HCD2, J403 NMJ6HCD2, J404 NMJ6HCD2, J405 Bypass FSW, J406 NMJ6HCD2, J407 Hold FSW, J408 OLED 0.91 128x32, K401 G6K-2F-Y, Q401 2N7002, Q402 2N7002, Q403 2N7002, SW101 100-DP6, SW102 100-DP6, SW103 100-DP6, U201 STM32H750VBT6, U202 W25Q128JVSIQ, U301 TPS54202DDC, U302 NCP718ASN500T1G, U401 MCP6001T-I/OT, U501 OPA2348AIDR, U601 THS4522IPW, U701 OPA2365AIDR, U702 OPA1688IDR, Y201 25MHz 9pF

Commit message: Update to 3v3 power layout
Parts:
- moved C306 15.2 mm to (123.2, 57.0)
- moved C305 6.62 mm to (141.0, 55.8), turned to -90 degrees
- moved L301 5.90 mm to (131.9, 57.0), turned to 180 degrees
- moved C307 3.75 mm to (126.8, 57.0)
- moved C304 3.46 mm to (137.7, 58.2)
- moved U301 3.46 mm to (137.7, 55.8)
Connections:
- net /ADC Driver/FDA_INN renamed Net-(U601A-INN)
- net /ADC Driver/FDA_INP renamed Net-(U601A-INP)
- net /ADC Driver/FDA_OUTN renamed Net-(U601A-OUTN)
- net /ADC Driver/FDA_OUTP renamed Net-(U601A-OUTP)
- net /ADC Driver/FDB_INN renamed Net-(U601B-INN)
- net /ADC Driver/FDB_INP renamed Net-(U601B-INP)
- net /ADC Driver/FDB_OUTN renamed Net-(U601B-OUTN)
- net /ADC Driver/FDB_OUTP renamed Net-(U601B-OUTP)
- net /Analog In and Out/IN_AC renamed Net-(U701A-+)
- net /Analog In and Out/IN_AC_R renamed Net-(U701B-+)
- net /Analog In and Out/IN_BUF_OUT renamed Net-(R703-Pad1)
- net /Analog In and Out/IN_BUF_OUT_R renamed Net-(U701B--)
- net /Analog In and Out/IN_FB renamed Net-(U701A--)
- net /Analog In and Out/IN_GAIN renamed Net-(C707-Pad1)
- net /Analog In and Out/OUTL_AC renamed Net-(C704-Pad2)
- net /Analog In and Out/OUTL_AMP renamed Net-(C704-Pad1)
- net /Analog In and Out/OUTL_N renamed Net-(U702A--)
- net /Analog In and Out/OUTL_P renamed Net-(U702A-+)
- net /Analog In and Out/OUTR_AC renamed Net-(C705-Pad2)
- net /Analog In and Out/OUTR_AMP renamed Net-(C705-Pad1)
- net /Analog In and Out/OUTR_N renamed Net-(U702B--)
- net /Analog In and Out/OUTR_P renamed Net-(U702B-+)
- net /Codec/PDN renamed Net-(IC501-PDN)
- net /Codec/VCOM renamed Net-(IC501-VCOM)
- net /Codec/VCOM_A_RAW renamed Net-(U501A--)
- net /Codec/VCOM_B_RAW renamed Net-(U501B--)
- net /Controls and LEDs/POT1_W renamed Net-(R101-Pad1)
- net /Controls and LEDs/POT2_W renamed Net-(R102-Pad1)
- net /Controls and LEDs/POT3_W renamed Net-(R103-Pad1)
- net /Controls and LEDs/POT5_W renamed Net-(R105-Pad1)
- net /Jacks and Bypass/EXP_BUF_IN renamed Net-(U401-+)
- net /Jacks and Bypass/EXP_BUF_OUT renamed Net-(U401--)
- net /Jacks and Bypass/EXP_RING renamed Net-(J406-PadR)
- net /Jacks and Bypass/EXP_TIP renamed Net-(D406-A2)
- net /Jacks and Bypass/FSW_BYPASS renamed Net-(J405-Pin_1)
- net /Jacks and Bypass/FSW_HOLD renamed Net-(J407-Pin_1)
- net /Jacks and Bypass/IN renamed Net-(D403-A2)
- net /Jacks and Bypass/LED_EFF_G renamed Net-(Q402-G)
- net /Jacks and Bypass/LED_EFF_K renamed Net-(D113-K)
- net /Jacks and Bypass/LED_EFF_LOW renamed Net-(Q402-D)
- net /Jacks and Bypass/LED_HOLD_G renamed Net-(Q403-G)
- net /Jacks and Bypass/LED_HOLD_K renamed Net-(D114-K)
- net /Jacks and Bypass/LED_HOLD_LOW renamed Net-(Q403-D)
- net /Jacks and Bypass/OUT_L renamed Net-(D404-A2)
- net /Jacks and Bypass/RELAY_COIL renamed Net-(D402-K)
- net /Jacks and Bypass/RELAY_G renamed Net-(Q401-G)
- net /Jacks and Bypass/RELAY_LOW renamed Net-(D402-A)
- net /MCU/BOOT0 renamed Net-(U201-BOOT0)
- net /MCU/HSE_IN renamed Net-(U201-PH0)
- net /MCU/HSE_OUT renamed Net-(U201-PH1)
- net /MCU/NRST renamed Net-(U201-NRST)
- net /MCU/QSPI_IO0 renamed Net-(U201-PE7)
- net /MCU/QSPI_IO1 renamed Net-(U201-PE8)
- net /MCU/QSPI_IO2 renamed Net-(U201-PE9)
- net /MCU/QSPI_IO3 renamed Net-(U201-PE10)
- net /MCU/SWCLK renamed Net-(U201-PA14)
- net /MCU/SWCLK_N renamed Net-(W201-SWCLK/TCK)
- net /MCU/SWDIO renamed Net-(U201-PA13)
- net /MCU/SWDIO_N renamed Net-(W201-SWDIO/TMS)
- net /MCU/SWO renamed Net-(U201-PB3)
- net /MCU/VCAP1 renamed Net-(C201-Pad1)
- net /MCU/VCAP2 renamed Net-(C202-Pad1)
- net /Power/BUCK_BOOT renamed Net-(U301-BOOT)
- net /Power/BUCK_FB renamed Net-(U301-FB)
- net /Power/BUCK_FBT renamed Net-(R301-Pad2)
- net /Power/DC_F renamed Net-(D302-A)
- net /Power/DC_IN renamed Net-(D301-A2)
- net /Power/LDO_IN renamed Net-(U302-EN)
- net /Power/LDO_OUT renamed Net-(U302-OUT)
- net /Power/SW renamed Net-(U301-SW)
Routing:
- net +3V3: track 310.7 -> 327.4 mm, vias 34 -> 33
- net Net-(U301-SW): track 16.1 -> 11.4 mm, vias 3 -> 2
- net Net-(U301-FB): track 10.6 -> 12.1 mm
- net +9V: track 238.1 -> 237.8 mm, vias 6 -> 5
