File: kicad/the_harp/The Harp.kicad_pcb (KiCad board)
At the start: 4 copper layers, 56 x 94.5 mm, 181 parts, among them IC501 AK4621EF, J401 PJ-063AH, J402 NMJ6HCD2, J403 NMJ6HCD2, J404 NMJ6HCD2, J405 Bypass FSW, J406 NMJ6HCD2, J407 Hold FSW, J408 OLED 0.91 128x32, K401 G6K-2F-Y, Q401 2N7002, Q402 2N7002, Q403 2N7002, SW101 100-DP6, SW102 100-DP6, SW103 100-DP6, U201 STM32H750VBT6, U202 W25Q128JVSIQ, U301 TPS54202DDC, U302 NCP718ASN500T1G, U401 MCP6001T-I/OT, U501 OPA2348AIDR, U601 THS4522IPW, U701 OPA2365AIDR, U702 OPA1688IDR, Y201 25MHz 9pF

Commit message: routing
Parts:
- moved R504 1.19 mm to (146.5, 79.9), turned to -90 degrees
Routing:
- net Net-(R102-Pad1): track 0.00 -> 28.2 mm, vias 0 -> 2
- net EFFECT_OUT_R: track 8.73 -> 32.8 mm
- net CODEC_CCLK: track 0.00 -> 11.0 mm, vias 0 -> 2
- net VCOM_A: track 75.9 -> 85.1 mm
- net CODEC_BICK: track 0.00 -> 5.31 mm, vias 0 -> 1
- net +3V3: track 344.4 -> 340.0 mm
- net Net-(U401-+): track 47.6 -> 50.8 mm
- net GND: track 120.2 -> 117.3 mm
- net CODEC_SDTO: track 13.2 -> 14.6 mm
- net Net-(Q401-G): track 26.9 -> 27.6 mm
- net EFFECT_IN_BUF_R: track 32.8 -> 33.4 mm
- net Net-(U501A--): track 5.45 -> 4.80 mm
- net CODEC_SDTI: track 11.1 -> 10.5 mm
- net Net-(IC501-VCOM): track 85.5 -> 86.1 mm
- net Net-(R101-Pad1): track 29.9 -> 29.4 mm
