File: kicad/the_harp/Jacks and Bypass.kicad_sch (KiCad schematic)
At the start: 38 parts, among them J402 NMJ6HCD2, J403 NMJ6HCD2, J404 NMJ6HCD2, J405 Bypass FSW, J406 NMJ6HCD2, J407 Hold FSW, K401 G6K-2F-Y, Q401 2N7002, Q402 2N7002, Q403 2N7002, U401 MCP6001T-I/OT

Commit message: Stereo single-ended input and an OLED display
IN becomes a TRS jack (tip left, ring right) with a second OPA2365 buffer and
THS4522 channel B into the AK4621EF's AINR; the codec inputs are no longer
parked. A mono plug is detected by the right channel reading silence. The
twelve note LEDs and R107-R118 give way to a 0.91 in I2C OLED connector (J408,
PB6/PB7) with 4.7k pull-ups. Schematic regenerated (190 parts, netlist OK on
all sheets); design brief, PCB plan, firmware requirements and the design
report updated. The PCB still carries the old LED footprints until Update PCB
from Schematic is run in KiCad.

Co-Authored-By: Claude Sonnet 5.5 <noreply@anthropic.com>
Claude-Session: https://claude.ai/code/session_016hDejPHPgG8auBLMyByYZK
Parts:
- added D407: PESD5V0U1BB,115, Diode_SMD:D_SOD-523, symbol Device:D_TVS
Connections:
- net GND: now also D407.1 (A1); no longer J402.R
- new net IN_R: D407.2 (A2), J402.R
Other:
- note added: "Jacks on the Alchemist positions: IN (J402, right lower), EXP (J406, right upper), OUT L (J403, left lower), OUT R (J404, left upper). Relay true bypass after The Alchemist: K401 (Omron G6K-2F-Y, 5 V coil) at rest joins IN to OUT L (2-3) and grounds the effect input (6-7); energised it routes IN to the effect (5-6) and the effect to OUT L (3-4). IN is a TRS jack, tip = left, ring = right: a mono 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"
- note removed: "Jacks on the Alchemist positions: IN (J402, right lower), EXP (J406, right upper), OUT L (J403, left lower), OUT R (J404, left upper). Relay true bypass after The Alchemist: K401 (Omron G6K-2F-Y, 5 V coil) at rest joins IN to OUT L (2-3) and grounds the effect input (6-7); energised it routes IN to the effect (5-6) and the effect to OUT L (3-4). IN jack ring to GND, as The Alchemist. OUT R is dri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"
